File: kicad/lcdclock.sch (KiCad schematic (older format))
At the start: 26 parts, among them J1 Conn_JLink_SWD, Q1 BSH205, SW1 SW_Push, U1 STM32L073xx_48, U2 ELV_DCF-2, U3 TPS70630, U4 LCD, Y1 32.768kHz 12.5pF

Commit message: Final fixes
Connections:
- net VCC: no longer C7.1, U1.1 (VLCD)
- new net: C7.1, U1.1 (VLCD)
Changed lines of the file:
@@
 Sheet 1 1
 Title "LCD Clock"
-Date "2017-09-18"
+Date ""
 Rev ""
 Comp ""
@@
 Wire Wire Line
 	6200 1050 6100 1050
-Wire Wire Line
-	6100 950  6100 1550
-Connection ~ 6100 1050
 $Comp
 L SW_Push SW1
@@
 $EndComp
 $Comp
-L VCC #PWR012
-U 1 1 59C307CF
-P 6100 950
-F 0 "#PWR012" H 6100 800 50  0001 C CNN
-F 1 "VCC" H 6100 1100 50  0000 C CNN
-F 2 "" H 6100 950 50  0001 C CNN
-F 3 "" H 6100 950 50  0001 C CNN
-	1    6100 950
-	1    0    0    -1
-$EndComp
-$Comp
 L VCC #PWR013
 U 1 1 59C30C48
@@
 Text Notes 8600 3900 0    60   ~ 0
 Backlight\nDo not connect if not needed.
+Wire Wire Line
+	6100 1050 6100 1550
 $EndSCHEMATC
